Commit message: adding moveit packages configs

File: install/ur5e_robot_config/share/ur5e_robot_config/urdf/my_gripper.xacro (robot description, xacro)
@@ -1,23 +1 @@
-<?xml version="1.0"?>
-<robot xmlns:xacro="http://ros.org/wiki/xacro">
-  <!-- Usage: <xacro:my_gripper parent="tool0"/> -->
-  <xacro:macro name="my_gripper" params="parent">
-    <link name="my_gripper_link">
-      <inertial><mass value="0.2"/><origin xyz="0 0 0"/><inertia ixx="1e-4" ixy="0" ixz="0" iyy="1e-4" iyz="0" izz="1e-4"/></inertial>
-      <visual><origin xyz="0 0 0.07"/><geometry><box size="0.03 0.03 0.14"/></geometry></visual>
-      <collision><origin xyz="0 0 0.07"/><geometry><box size="0.03 0.03 0.14"/></geometry></collision>
-    </link>
-    <joint name="my_gripper_joint" type="fixed">
-      <parent link="${parent}"/>
-      <child  link="my_gripper_link"/>
-      <origin xyz="0 0 0" rpy="0 0 0"/>
-    </joint>
-    <!-- Define TCP at the gripper tip -->
-    <link name="tcp"/>
-    <joint name="tcp_fixed" type="fixed">
-      <parent link="my_gripper_link"/>
-      <child  link="tcp"/>
-      <origin xyz="0 0 0.14" rpy="0 0 0"/>
-    </joint>
-  </xacro:macro>
-</robot>
+/home/ryanl/4231/MTRN4231_Project/src/ur5e_robot_config/urdf/my_gripper.xacro

File: install/ur5e_robot_config/share/ur5e_robot_config/urdf/ur5e_with_tool.urdf.xacro (robot description, xacro)
@@ -1,22 +1 @@
-<?xml version="1.0"?>
-<robot name="ur5e_with_tool" xmlns:xacro="http://ros.org/wiki/xacro">
-  <!-- Vendor UR description -->
-  <xacro:include filename="$(find ur_description)/urdf/ur.urdf.xacro"/>
-  <!-- Our simple tool -->
-  <xacro:include filename="$(find ur5e_robot_moveit)/urdf/my_gripper.xacro"/>
-  <!-- If you have a real calibration file later, set its path via a param -->
-  <xacro:arg name="kinematics_parameters_file" default=""/>
-  <!-- Build the robot -->
-  <xacro:ur_robot
-      name:="ur5e"
-      ur_type:="ur5e"
-      prefix:=""
-      safety_limits:="true"
-      safety_pos_margin:="0.15"
-      safety_k_position:="20"
-      kinematics_parameters_file:="${kinematics_parameters_file}"
-      >
-    <!-- Attach our gripper to tool0; expose a TCP link named 'tcp' -->
-    <xacro:my_gripper parent="tool0"/>
-  </xacro:ur_robot>
-</robot>
+/home/ryanl/4231/MTRN4231_Project/src/ur5e_robot_config/urdf/ur5e_with_tool.urdf.xacro
