Commit message: rviz working

File: src/arm_controller/urdf/ur5e_with_tool.urdf.xacro (robot description, xacro)
@@ -1,24 +1,48 @@
 <?xml version="1.0"?>
-<robot name="ur5e_with_tool" xmlns:xacro="http://www.ros.org/wiki/xacro">
+<robot xmlns:xacro="http://www.ros.org/wiki/xacro" name="ur5e_with_tool">
+  <!-- Define PROPERTIES so the vendor xacro sees them BEFORE include -->
+  <xacro:property name="name"    value="ur5e"/>
+  <xacro:property name="ur_type" value="ur5e"/>
+  <!-- Other knobs as properties -->
+  <xacro:property name="prefix" value=""/>
+  <xacro:property name="use_fake_hardware" value="true"/>
+  <xacro:property name="robot_ip" value=""/>
+  <xacro:property name="kinematics_parameters_file" value=""/>
+  <xacro:property name="visual_parameters_file"     value=""/>
+  <!-- Include UR vendor macros (Humble supports $(find ...)) -->
   <xacro:include filename="$(find ur_description)/urdf/ur.urdf.xacro"/>
+  <!-- Instantiate the macro (NORMAL XML attributes; no ':=') -->
   <xacro:ur_robot
-      name="ur5e"
-      ur_type="ur5e"
-      prefix=""
-      joint_limited="false"
+      name="${name}"
+      ur_type="${ur_type}"
+      prefix="${prefix}"
+      use_fake_hardware="${use_fake_hardware}"
+      robot_ip="${robot_ip}"
       safety_limits="true"
       safety_pos_margin="0.15"
       safety_k_position="20"
-      use_fake_hardware="true"
-      kinematics_params_file="$(find ur_description)/config/ur5e/default_kinematics.yaml"
-      visual_parameters_config_file="$(find ur_description)/config/ur5e/visual_parameters.yaml">
-    <origin xyz="0 0 0" rpy="0 0 0"/>
+      kinematics_parameters_file="${kinematics_parameters_file}"
+      visual_parameters_file="${visual_parameters_file}">
+    <!-- simple fixed box as the gripper attached to tool0 -->
+    <link name="simple_gripper_link">
+      <visual>
+        <geometry><box size="0.04 0.04 0.10"/></geometry>
+        <origin xyz="0 0 0.05" rpy="0 0 0"/>
+      </visual>
+      <collision>
+        <geometry><box size="0.04 0.04 0.10"/></geometry>
+        <origin xyz="0 0 0.05" rpy="0 0 0"/>
+      </collision>
+      <inertial>
+        <origin xyz="0 0 0.05" rpy="0 0 0"/>
+        <mass value="0.2"/>
+        <inertia ixx="1e-4" iyy="1e-4" izz="1e-4" ixy="0" ixz="0" iyz="0"/>
+      </inertial>
+    </link>
+    <joint name="tool0_to_gripper" type="fixed">
+      <parent link="${prefix}tool0"/>
+      <child  link="simple_gripper_link"/>
+      <origin xyz="0 0 0" rpy="0 0 0"/>
+    </joint>
   </xacro:ur_robot>
-  <!-- Your TCP -->
-  <link name="tool0"/>
-  <joint name="wrist_3_to_tool0" type="fixed">
-    <parent link="wrist_3_link"/>
-    <origin xyz="0.10 0 0" rpy="0 -1.57079632679 0"/>
-    <child link="tool0"/>
-  </joint>
 </robot>

Commit message: fixing controller

File: src/arm_controller/urdf/ur5e_with_tool.urdf.xacro (robot description, xacro)
@@ -1,48 +1,57 @@
 <?xml version="1.0"?>
-<robot xmlns:xacro="http://www.ros.org/wiki/xacro" name="ur5e_with_tool">
-  <!-- Define PROPERTIES so the vendor xacro sees them BEFORE include -->
-  <xacro:property name="name"    value="ur5e"/>
-  <xacro:property name="ur_type" value="ur5e"/>
-  <!-- Other knobs as properties -->
-  <xacro:property name="prefix" value=""/>
-  <xacro:property name="use_fake_hardware" value="true"/>
-  <xacro:property name="robot_ip" value=""/>
-  <xacro:property name="kinematics_parameters_file" value=""/>
-  <xacro:property name="visual_parameters_file"     value=""/>
-  <!-- Include UR vendor macros (Humble supports $(find ...)) -->
+<robot name="ur5e" xmlns:xacro="http://www.ros.org/wiki/xacro">
+  <!-- args expected by ur_description -->
+  <xacro:arg name="name"                 default="ur5e"/>
+  <xacro:arg name="ur_type"              default="ur5e"/>
+  <xacro:arg name="use_fake_hardware"    default="true"/>
+  <xacro:arg name="prefix"               default=""/>
+  <xacro:arg name="visual_parameters_file"
+             default="/opt/ros/humble/share/ur_description/config/ur5/visual_parameters.yaml"/>
+  <!-- bring in the official UR model -->
   <xacro:include filename="$(find ur_description)/urdf/ur.urdf.xacro"/>
-  <!-- Instantiate the macro (NORMAL XML attributes; no ':=') -->
   <xacro:ur_robot
-      name="${name}"
-      ur_type="${ur_type}"
-      prefix="${prefix}"
-      use_fake_hardware="${use_fake_hardware}"
-      robot_ip="${robot_ip}"
-      safety_limits="true"
-      safety_pos_margin="0.15"
-      safety_k_position="20"
-      kinematics_parameters_file="${kinematics_parameters_file}"
-      visual_parameters_file="${visual_parameters_file}">
-    <!-- simple fixed box as the gripper attached to tool0 -->
-    <link name="simple_gripper_link">
-      <visual>
-        <geometry><box size="0.04 0.04 0.10"/></geometry>
-        <origin xyz="0 0 0.05" rpy="0 0 0"/>
-      </visual>
-      <collision>
-        <geometry><box size="0.04 0.04 0.10"/></geometry>
-        <origin xyz="0 0 0.05" rpy="0 0 0"/>
-      </collision>
-      <inertial>
-        <origin xyz="0 0 0.05" rpy="0 0 0"/>
-        <mass value="0.2"/>
-        <inertia ixx="1e-4" iyy="1e-4" izz="1e-4" ixy="0" ixz="0" iyz="0"/>
-      </inertial>
-    </link>
-    <joint name="tool0_to_gripper" type="fixed">
-      <parent link="${prefix}tool0"/>
-      <child  link="simple_gripper_link"/>
-      <origin xyz="0 0 0" rpy="0 0 0"/>
-    </joint>
-  </xacro:ur_robot>
+      name="$(arg name)"
+      ur_type="$(arg ur_type)"
+      prefix="$(arg prefix)"
+      kinematics_parameters_file=""
+      physical_parameters_file=""
+      visual_parameters_file="$(arg visual_parameters_file)"
+      transmission_hw_interface="hardware_interface/PositionJointInterface"
+      use_fake_hardware="$(arg use_fake_hardware)"
+      safety_limits="false" safety_pos_margin="0.0" safety_k_position="0.0" />
+  <!-- === End-effector: simple block mounted on tool0 === -->
+  <link name="${prefix}ee_adapter"/>
+  <joint name="${prefix}tool0_to_ee_adapter" type="fixed">
+    <parent link="${prefix}tool0"/>
+    <child  link="${prefix}ee_adapter"/>
+    <origin xyz="0 0 0.0" rpy="0 0 0"/>
+  </joint>
+  <link name="${prefix}gripper_base">
+    <visual>
+      <origin xyz="0 0 0.08" rpy="0 0 0"/>
+      <geometry><box size="0.04 0.06 0.16"/></geometry>
+      <material name="gray"><color rgba="0.7 0.7 0.7 1.0"/></material>
+    </visual>
+    <collision>
+      <origin xyz="0 0 0.08" rpy="0 0 0"/>
+      <geometry><box size="0.04 0.06 0.16"/></geometry>
+    </collision>
+    <inertial>
+      <origin xyz="0 0 0.08" rpy="0 0 0"/>
+      <mass value="0.5"/>
+      <inertia ixx="0.001" ixy="0" ixz="0" iyy="0.001" iyz="0" izz="0.001"/>
+    </inertial>
+  </link>
+  <joint name="${prefix}ee_adapter_to_gripper" type="fixed">
+    <parent link="${prefix}ee_adapter"/>
+    <child  link="${prefix}gripper_base"/>
+    <origin xyz="0 0 0.0" rpy="0 0 0"/>
+  </joint>
+  <!-- Optional TCP alias a bit below the block tip -->
+  <link name="${prefix}tcp_link"/>
+  <joint name="${prefix}gripper_to_tcp" type="fixed">
+    <parent link="${prefix}gripper_base"/>
+    <child  link="${prefix}tcp_link"/>
+    <origin xyz="0 0 0.18" rpy="0 0 0"/>
+  </joint>
 </robot>

Commit message: still getting endeffector showing up on the robot

File: src/arm_controller/urdf/ur5e_with_tool.urdf.xacro (robot description, xacro)
@@ -1,52 +1,17 @@
 <?xml version="1.0"?>
-<robot name="ur5e" xmlns:xacro="http://www.ros.org/wiki/xacro">
-  <!-- args -->
-  <xacro:arg name="name"              default="ur5e"/>
-  <xacro:arg name="use_fake_hardware" default="true"/>
-  <xacro:arg name="prefix"            default=""/>
-  <xacro:arg name="visual_parameters_file"
-             default="/opt/ros/humble/share/ur_description/config/ur5/visual_parameters.yaml"/>
-  <!-- Bring in UR5e-specific xacro and instantiate it (NO ur_type arg) -->
-  <xacro:include filename="$(find ur_description)/urdf/ur5e.urdf.xacro"/>
-  <xacro:ur5e_robot
-      name="$(arg name)"
-      prefix="$(arg prefix)"
-      visual_parameters_file="$(arg visual_parameters_file)"
-      use_fake_hardware="$(arg use_fake_hardware)"
-      safety_limits="false" safety_pos_margin="0.0" safety_k_position="0.0" />
-  <!-- === Simple EE mounted at tool0 === -->
-  <link name="${prefix}ee_adapter"/>
-  <joint name="${prefix}tool0_to_ee_adapter" type="fixed">
-    <parent link="${prefix}tool0"/>
-    <child  link="${prefix}ee_adapter"/>
-    <origin xyz="0 0 0.0" rpy="0 0 0"/>
-  </joint>
-  <link name="${prefix}gripper_base">
-    <visual>
-      <origin xyz="0 0 0.08" rpy="0 0 0"/>
-      <geometry><box size="0.04 0.06 0.16"/></geometry>
-      <material name="gray"><color rgba="0.7 0.7 0.7 1.0"/></material>
-    </visual>
-    <collision>
-      <origin xyz="0 0 0.08" rpy="0 0 0"/>
-      <geometry><box size="0.04 0.06 0.16"/></geometry>
-    </collision>
-    <inertial>
-      <origin xyz="0 0 0.08" rpy="0 0 0"/>
-      <mass value="0.5"/>
-      <inertia ixx="0.001" ixy="0" ixz="0" iyy="0.001" iyz="0" izz="0.001"/>
-    </inertial>
-  </link>
-  <joint name="${prefix}ee_adapter_to_gripper" type="fixed">
-    <parent link="${prefix}ee_adapter"/>
-    <child  link="${prefix}gripper_base"/>
-    <origin xyz="0 0 0.0" rpy="0 0 0"/>
-  </joint>
-  <!-- TCP alias (tip) -->
-  <link name="${prefix}tcp_link"/>
-  <joint name="${prefix}gripper_to_tcp" type="fixed">
-    <parent link="${prefix}gripper_base"/>
-    <child  link="${prefix}tcp_link"/>
-    <origin xyz="0 0 0.18" rpy="0 0 0"/>
+<robot name="ur5e_with_tool" xmlns:xacro="http://www.ros.org/wiki/xacro">
+  <!-- Required args so ur_description's xacro doesn't error -->
+  <xacro:arg name="name" default="ur"/>
+  <xacro:arg name="ur_type" default="ur5e"/>
+  <!-- UR5e -->
+  <xacro:include filename="$(find ur_description)/urdf/ur.urdf.xacro"/>
+  <!-- End effector (your package + URDF) -->
+  <xacro:include filename="$(find end_effector_description)/urdf/end_effector.urdf"/>
+  <!-- Coupler joint: tool0 -> ee_mount (rename child if your root link differs) -->
+  <joint name="ee_coupler_joint" type="fixed">
+    <parent link="tool0"/>
+    <child  link="ee_mount"/>
+    <!-- Adjust if your STL needs an offset/rotation relative to tool0 -->
+    <origin xyz="0 0 0.10" rpy="0 ${pi} 0"/>
   </joint>
 </robot>

File: src/end_effector_description/urdf/end_effector.xacro (robot description, xacro)
@@ -1,11 +1,19 @@
 <?xml version="1.0"?>
-<robot name="end_effector_standalone" xmlns:xacro="http://www.ros.org/wiki/xacro">
-  <!-- Humble: $(find ...) is OK -->
-  <xacro:include filename="$(find end_effector_description)/urdf/end_effector.urdf.xacro"/>
-  <!-- Dummy base to view it alone -->
-  <link name="ee_root_link"/>
-  <!-- Instantiate the macro (prefix is defined here!) -->
-  <xacro:end_effector prefix="" parent="ee_root_link">
-    <origin xyz="0 0 0" rpy="0 0 0"/>
-  </xacro:end_effector>
+<robot name="end_effector" xmlns:xacro="http://ros.org/wiki/xacro">
+  <!-- optional args if you want to tune offsets/scales -->
+  <xacro:arg name="mesh_scale" default="0.001 0.001 0.001"/>
+  <xacro:arg name="mount_to_mesh_xyz" default="0 0 0"/>
+  <xacro:arg name="mount_to_mesh_rpy" default="0 0 0"/>
+  <xacro:macro name="end_effector" params="">
+    <link name="ee_mount">
+      <visual>
+        <origin xyz="${mount_to_mesh_xyz}" rpy="${mount_to_mesh_rpy}"/>
+        <geometry>
+          <mesh filename="package://end_effector_description/meshes/claw_assembly.stl"
+                scale="${mesh_scale}"/>
+        </geometry>
+      </visual>
+    </link>
+    <!-- add extra links/joints later if you split the mesh -->
+  </xacro:macro>
 </robot>
