Commit message: working ish

File: install/end_effector_description/share/end_effector_description/urdf/end_effector.xacro (robot description, xacro)
@@ -1 +1,19 @@
-/home/ryanl/4231/MTRN4231_Project/src/end_effector_description/urdf/end_effector.xacro
+<?xml version="1.0"?>
+<robot name="end_effector" xmlns:xacro="http://ros.org/wiki/xacro">
+  <!-- optional args if you want to tune offsets/scales -->
+  <xacro:arg name="mesh_scale" default="0.001 0.001 0.001"/>
+  <xacro:arg name="mount_to_mesh_xyz" default="0 0 0"/>
+  <xacro:arg name="mount_to_mesh_rpy" default="0 0 0"/>
+  <xacro:macro name="end_effector" params="">
+    <link name="ee_mount">
+      <visual>
+        <origin xyz="${mount_to_mesh_xyz}" rpy="${mount_to_mesh_rpy}"/>
+        <geometry>
+          <mesh filename="package://end_effector_description/meshes/claw_assembly.stl"
+                scale="${mesh_scale}"/>
+        </geometry>
+      </visual>
+    </link>
+    <!-- add extra links/joints later if you split the mesh -->
+  </xacro:macro>
+</robot>
