Commit message: made a setup assitance to generate moveit config

File: install/end_effector_description/share/end_effector_description/urdf/end_effector.urdf.xacro (robot description, xacro)
@@ -16,5 +16,5 @@
       <!-- Use a simple box for collision (faster & more robust than STL) -->
       <collision>
-        <origin xyz="0 0 0" rpy="0 0 0"/>
+        <origin xyz="0.00 0.00 0.02" rpy="0 0 0"/>
         <geometry>
           <!-- tune these to roughly bound your gripper -->

File: install/end_effector_description/share/end_effector_description/urdf/end_effector_withDriverSupport.xacro (robot description, xacro)
@@ -9,4 +9,5 @@
   <!-- Don't pass ur_type here; it's consumed internally by ur.urdf.xacro -->
   <!-- <xacro:ur_robot name="$(arg name)"/> -->
+  <!-- <xacro:ur_robot name="$(arg name)"/> -->
   <!-- End-effector macro (your file above) -->
   <xacro:include filename="$(find end_effector_description)/urdf/end_effector.urdf.xacro"/>
