Commit message: wsl doesn't work for setup assistant

File: install/arm_controller/share/arm_controller/urdf/ur5e_with_tool.urdf.xacro (robot description, xacro)
@@ -1,17 +1 @@
-<?xml version="1.0"?>
-<robot name="ur5e_with_tool" xmlns:xacro="http://www.ros.org/wiki/xacro">
-  <!-- Required args so ur_description's xacro doesn't error -->
-  <xacro:arg name="name" default="ur"/>
-  <xacro:arg name="ur_type" default="ur5e"/>
-  <!-- UR5e -->
-  <xacro:include filename="$(find ur_description)/urdf/ur.urdf.xacro"/>
-  <!-- End effector (your package + URDF) -->
-  <xacro:include filename="$(find end_effector_description)/urdf/end_effector.urdf"/>
-  <!-- Coupler joint: tool0 -> ee_mount (rename child if your root link differs) -->
-  <joint name="ee_coupler_joint" type="fixed">
-    <parent link="tool0"/>
-    <child  link="ee_mount"/>
-    <!-- Adjust if your STL needs an offset/rotation relative to tool0 -->
-    <origin xyz="0 0 0.10" rpy="0 ${pi} 0"/>
-  </joint>
-</robot>
+/home/ryanl/4231/MTRN4231_Project/src/arm_controller/urdf/ur5e_with_tool.urdf.xacro

File: install/ur5e_custom_description/share/ur5e_custom_description/urdf/ur5e_with_tool.urdf.xacro (robot description, xacro)
@@ -1,44 +1 @@
-<?xml version="1.0"?>
-<robot name="ur5e_with_tool" xmlns:xacro="http://www.ros.org/wiki/xacro">
-  <!-- ====== Common wrapper args (mirror your current wrapper) ====== -->
-  <xacro:arg name="name" default="ur"/>
-  <xacro:arg name="ur_type" default="ur5e"/>
-  <!-- UR config file args (same names you were passing in launch) -->
-  <xacro:arg name="joint_limit_params" default="$(find ur_description)/config/ur5e/joint_limits.yaml"/>
-  <xacro:arg name="kinematics_params"  default="$(find ur_description)/config/ur5e/default_kinematics.yaml"/>
-  <xacro:arg name="physical_params"    default="$(find ur_description)/config/ur5e/physical_parameters.yaml"/>
-  <xacro:arg name="visual_params"      default="$(find ur_description)/config/ur5e/visual_parameters.yaml"/>
-  <!-- safety params (same names) -->
-  <xacro:arg name="safety_limits"     default="true"/>
-  <xacro:arg name="safety_pos_margin" default="0.15"/>
-  <xacro:arg name="safety_k_position" default="20"/>
-  <!-- (Optional, ignored by UR xacro, kept for compatibility) -->
-  <xacro:arg name="robot_ip" default="192.168.0.100"/>
-  <!-- ====== Include the UR base (from ur_description) ====== -->
-  <xacro:include filename="$(find ur_description)/urdf/ur.urdf.xacro"/>
-  <xacro:ur_robot
-      name="${name}"
-      ur_type="${ur_type}"
-      joint_limit_params="${joint_limit_params}"
-      kinematics_params="${kinematics_params}"
-      physical_params="${physical_params}"
-      visual_params="${visual_params}"
-      safety_limits="${safety_limits}"
-      safety_pos_margin="${safety_pos_margin}"
-      safety_k_position="${safety_k_position}"
-  />
-  <!-- ====== Include your end effector ====== -->
-  <!-- If your EE lives in a separate package, keep this include: -->
-  <xacro:include filename="$(find end_effector_description)/urdf/end_effector.urdf"/>
-  <!-- If your EE xacro defines a known root link (e.g., 'ee_body'), keep it here.
-       Otherwise, change ee_root_link's default to your actual EE root link. -->
-  <!-- <xacro:arg name="ee_root_link" default="ee_body"/> -->
-  <!-- ====== Mount: UR 'tool0' -> EE root link ====== -->
-  <!-- Coupler joint: tool0 -> ee_mount (rename child if your root link differs) -->
-  <joint name="ee_coupler_joint" type="fixed">
-    <parent link="tool0"/>
-    <child  link="ee_mount"/>
-    <!-- Adjust if your STL needs an offset/rotation relative to tool0 -->
-    <origin xyz="0 0 0.10" rpy="0 ${pi} 0"/>
-  </joint>
-</robot>
+/home/ryanl/4231/MTRN4231_Project/src/ur5e_custom_description/urdf/ur5e_with_tool.urdf.xacro

File: src/end_effector_description/urdf/end_effector.urdf.xacro (robot description, xacro)
@@ -1,35 +1,45 @@
 <?xml version="1.0"?>
-<robot name="claw_end_effector" xmlns:xacro="http://ros.org/wiki/xacro">
-  <!-- mm → m scale -->
-  <xacro:property name="scale" value="0.001"/>
-  <!-- Simple mass/inertia placeholders (tune later) -->
-  <xacro:property name="m" value="0.5"/>
-  <xacro:property name="I" value="1.0"/>
-  <!-- Macro: a single mesh link and a fixed joint to its parent -->
-  <xacro:macro name="end_effector" params="prefix parent">
-    <link name="${prefix}claw">
+<robot name="end_effector" xmlns:xacro="http://ros.org/wiki/xacro">
+  <!-- Constants -->
+  <xacro:property name="scale_factor" value="0.001"/>
+  <xacro:property name="mass_value" value="0.5"/>
+  <xacro:property name="inertia_value" value="1.0"/>
+  <!-- Helper: mesh link with inertial -->
+  <xacro:macro name="add_mesh_link" params="link_name mesh_path">
+    <link name="${link_name}">
       <visual>
+        <origin xyz="0 0 0" rpy="0 0 0"/>
         <geometry>
-          <mesh filename="package://end_effector_description/meshes/claw_assembly.stl"
-                scale="${scale} ${scale} ${scale}"/>
+          <mesh filename="${mesh_path}" scale="${scale_factor} ${scale_factor} ${scale_factor}"/>
         </geometry>
       </visual>
+      <!-- Use a simple box for collision (faster & more robust than STL) -->
       <collision>
+        <origin xyz="0 0 0" rpy="0 0 0"/>
         <geometry>
-          <mesh filename="package://end_effector_description/meshes/claw_assembly.stl"
-                scale="${scale} ${scale} ${scale}"/>
+          <!-- tune these to roughly bound your gripper -->
+          <box size="0.06 0.09 0.11"/>
         </geometry>
       </collision>
       <inertial>
-        <mass value="${m}"/>
-        <inertia ixx="${I}" iyy="${I}" izz="${I}" ixy="0" ixz="0" iyz="0"/>
+        <origin xyz="0 0 0" rpy="0 0 0"/>
+        <mass value="${mass_value}"/>
+        <inertia ixx="${inertia_value}" ixy="0" ixz="0"
+                 iyy="${inertia_value}" iyz="0"
+                 izz="${inertia_value}"/>
       </inertial>
     </link>
-    <!-- Mount (adjust pose to suit your CAD) -->
-    <joint name="${prefix}mount_joint" type="fixed">
+  </xacro:macro>
+  <!-- Main end-effector macro -->
+  <xacro:macro name="end_effector" params="prefix parent">
+    <xacro:add_mesh_link
+      link_name="${prefix}gripper"
+      mesh_path="package://end_effector_description/meshes/claw_assembly.stl"/>
+    <!-- Mount to the parent (e.g., tool0). Adjust pose to suit your CAD. -->
+    <joint name="${prefix}gripper_mount" type="fixed">
       <parent link="${parent}"/>
-      <child  link="${prefix}claw"/>
-      <!-- Example: 110 mm forward, flip 180° about Y -->
-      <origin xyz="0 0 0.11" rpy="0 ${pi} 0"/>
+      <child  link="${prefix}gripper"/>
+      <!-- Example pose: 67 mm forward, rotate as needed -->
+      <origin xyz="0 0 0.067" rpy="0 ${pi} 0"/>
     </joint>
   </xacro:macro>

File: src/end_effector_description/urdf/end_effector_only.urdf.xacro (robot description, xacro)
@@ -1,6 +1,11 @@
-<?xml version="1.0"?>
+<?xml version="1.0" ?>
+<!-- Only displays the end-effector -->
 <robot name="end_effector_only" xmlns:xacro="http://ros.org/wiki/xacro">
-  <xacro:include filename="$(find end_effector_description)/urdf/end_effector.urdf.xacro"/>
-  <link name="ee_root_link"/>
-  <xacro:end_effector prefix="ee_" parent="ee_root_link"/>
+  <!-- Including the claw.urdf.xacro file to give scope to xacro:claw. Inclusion is a simple copy-and-paste of code. -->
+  <xacro:include filename="$(find end_effector_description)/urdf/end_effector.urdf.xacro" />
+  <!-- This is the abstract link which the base of the claw attaches to. -->
+  <link name="end_effector_root_link"/>
+  <!-- Instantiate the claw by using its macro. -->
+  <xacro:end_effector prefix="end_effector" parent="end_effector_root_link" >
+  </xacro:end_effector>
 </robot>

Commit message: just missing one step for setup assissant

File: install/arm_controller/share/arm_controller/urdf/ur5e_with_tool.urdf.xacro (robot description, xacro)
@@ -1 +1,17 @@
-/home/ryanl/4231/MTRN4231_Project/src/arm_controller/urdf/ur5e_with_tool.urdf.xacro
+<?xml version="1.0"?>
+<robot name="ur5e_with_tool" xmlns:xacro="http://www.ros.org/wiki/xacro">
+  <!-- Required args so ur_description's xacro doesn't error -->
+  <xacro:arg name="name" default="ur"/>
+  <xacro:arg name="ur_type" default="ur5e"/>
+  <!-- UR5e -->
+  <xacro:include filename="$(find ur_description)/urdf/ur.urdf.xacro"/>
+  <!-- End effector (your package + URDF) -->
+  <xacro:include filename="$(find end_effector_description)/urdf/end_effector.urdf"/>
+  <!-- Coupler joint: tool0 -> ee_mount (rename child if your root link differs) -->
+  <joint name="ee_coupler_joint" type="fixed">
+    <parent link="tool0"/>
+    <child  link="ee_mount"/>
+    <!-- Adjust if your STL needs an offset/rotation relative to tool0 -->
+    <origin xyz="0 0 0.10" rpy="0 ${pi} 0"/>
+  </joint>
+</robot>

File: install/end_effector_description/share/end_effector_description/urdf/end_effector.urdf.xacro (robot description, xacro)
@@ -1 +1,46 @@
-/home/ryanl/4231/MTRN4231_Project/src/end_effector_description/urdf/end_effector.urdf.xacro
+<?xml version="1.0"?>
+<robot name="end_effector" xmlns:xacro="http://ros.org/wiki/xacro">
+  <!-- Constants -->
+  <xacro:property name="scale_factor" value="0.001"/>
+  <xacro:property name="mass_value" value="0.5"/>
+  <xacro:property name="inertia_value" value="1.0"/>
+  <!-- Helper: mesh link with inertial -->
+  <xacro:macro name="add_mesh_link" params="link_name mesh_path">
+    <link name="${link_name}">
+      <visual>
+        <origin xyz="0 0 0" rpy="0 0 0"/>
+        <geometry>
+          <mesh filename="${mesh_path}" scale="${scale_factor} ${scale_factor} ${scale_factor}"/>
+        </geometry>
+      </visual>
+      <!-- Use a simple box for collision (faster & more robust than STL) -->
+      <collision>
+        <origin xyz="0 0 0" rpy="0 0 0"/>
+        <geometry>
+          <!-- tune these to roughly bound your gripper -->
+          <box size="0.06 0.09 0.11"/>
+        </geometry>
+      </collision>
+      <inertial>
+        <origin xyz="0 0 0" rpy="0 0 0"/>
+        <mass value="${mass_value}"/>
+        <inertia ixx="${inertia_value}" ixy="0" ixz="0"
+                 iyy="${inertia_value}" iyz="0"
+                 izz="${inertia_value}"/>
+      </inertial>
+    </link>
+  </xacro:macro>
+  <!-- Main end-effector macro -->
+  <xacro:macro name="end_effector" params="prefix parent">
+    <xacro:add_mesh_link
+      link_name="${prefix}gripper"
+      mesh_path="package://end_effector_description/meshes/claw_assembly.stl"/>
+    <!-- Mount to the parent (e.g., tool0). Adjust pose to suit your CAD. -->
+    <joint name="${prefix}gripper_mount" type="fixed">
+      <parent link="${parent}"/>
+      <child  link="${prefix}gripper"/>
+      <!-- Example pose: 67 mm forward, rotate as needed -->
+      <origin xyz="0 0 0.067" rpy="0 ${pi} 0"/>
+    </joint>
+  </xacro:macro>
+</robot>

File: install/end_effector_description/share/end_effector_description/urdf/end_effector_only.urdf.xacro (robot description, xacro)
@@ -1 +1,11 @@
-/home/ryanl/4231/MTRN4231_Project/src/end_effector_description/urdf/end_effector_only.urdf.xacro
+<?xml version="1.0" ?>
+<!-- Only displays the end-effector -->
+<robot name="end_effector_only" xmlns:xacro="http://ros.org/wiki/xacro">
+  <!-- Including the claw.urdf.xacro file to give scope to xacro:claw. Inclusion is a simple copy-and-paste of code. -->
+  <xacro:include filename="$(find end_effector_description)/urdf/end_effector.urdf.xacro" />
+  <!-- This is the abstract link which the base of the claw attaches to. -->
+  <link name="end_effector_root_link"/>
+  <!-- Instantiate the claw by using its macro. -->
+  <xacro:end_effector prefix="end_effector" parent="end_effector_root_link" >
+  </xacro:end_effector>
+</robot>

File: install/end_effector_description/share/end_effector_description/urdf/end_effector_withDriverSupport.xacro (robot description, xacro)
@@ -1 +1,15 @@
-/home/ryanl/4231/MTRN4231_Project/src/end_effector_description/urdf/end_effector_withDriverSupport.xacro
+<?xml version="1.0"?>
+<robot name="end_effector_withDriverSupport" xmlns:xacro="http://ros.org/wiki/xacro">
+  <!-- UR args (prefer ur5e unless you truly have ur5) -->
+  <xacro:arg name="name"    default="ur5e"/>
+  <xacro:arg name="ur_type" default="ur5"/>
+  <xacro:arg name="prefix"  default=""/>
+  <!-- UR robot -->
+  <xacro:include filename="$(find ur_description)/urdf/ur.urdf.xacro"/>
+  <!-- Don't pass ur_type here; it's consumed internally by ur.urdf.xacro -->
+  <!-- <xacro:ur_robot name="$(arg name)"/> -->
+  <!-- End-effector macro (your file above) -->
+  <xacro:include filename="$(find end_effector_description)/urdf/end_effector.urdf.xacro"/>
+  <!-- Mount the gripper to tool0 -->
+  <xacro:end_effector prefix="" parent="tool0"/>
+</robot>

File: install/ur5e_custom_description/share/ur5e_custom_description/urdf/ur5e_with_tool.urdf.xacro (robot description, xacro)
@@ -1 +1,44 @@
-/home/ryanl/4231/MTRN4231_Project/src/ur5e_custom_description/urdf/ur5e_with_tool.urdf.xacro
+<?xml version="1.0"?>
+<robot name="ur5e_with_tool" xmlns:xacro="http://www.ros.org/wiki/xacro">
+  <!-- ====== Common wrapper args (mirror your current wrapper) ====== -->
+  <xacro:arg name="name" default="ur"/>
+  <xacro:arg name="ur_type" default="ur5e"/>
+  <!-- UR config file args (same names you were passing in launch) -->
+  <xacro:arg name="joint_limit_params" default="$(find ur_description)/config/ur5e/joint_limits.yaml"/>
+  <xacro:arg name="kinematics_params"  default="$(find ur_description)/config/ur5e/default_kinematics.yaml"/>
+  <xacro:arg name="physical_params"    default="$(find ur_description)/config/ur5e/physical_parameters.yaml"/>
+  <xacro:arg name="visual_params"      default="$(find ur_description)/config/ur5e/visual_parameters.yaml"/>
+  <!-- safety params (same names) -->
+  <xacro:arg name="safety_limits"     default="true"/>
+  <xacro:arg name="safety_pos_margin" default="0.15"/>
+  <xacro:arg name="safety_k_position" default="20"/>
+  <!-- (Optional, ignored by UR xacro, kept for compatibility) -->
+  <xacro:arg name="robot_ip" default="192.168.0.100"/>
+  <!-- ====== Include the UR base (from ur_description) ====== -->
+  <xacro:include filename="$(find ur_description)/urdf/ur.urdf.xacro"/>
+  <xacro:ur_robot
+      name="${name}"
+      ur_type="${ur_type}"
+      joint_limit_params="${joint_limit_params}"
+      kinematics_params="${kinematics_params}"
+      physical_params="${physical_params}"
+      visual_params="${visual_params}"
+      safety_limits="${safety_limits}"
+      safety_pos_margin="${safety_pos_margin}"
+      safety_k_position="${safety_k_position}"
+  />
+  <!-- ====== Include your end effector ====== -->
+  <!-- If your EE lives in a separate package, keep this include: -->
+  <xacro:include filename="$(find end_effector_description)/urdf/end_effector.urdf"/>
+  <!-- If your EE xacro defines a known root link (e.g., 'ee_body'), keep it here.
+       Otherwise, change ee_root_link's default to your actual EE root link. -->
+  <!-- <xacro:arg name="ee_root_link" default="ee_body"/> -->
+  <!-- ====== Mount: UR 'tool0' -> EE root link ====== -->
+  <!-- Coupler joint: tool0 -> ee_mount (rename child if your root link differs) -->
+  <joint name="ee_coupler_joint" type="fixed">
+    <parent link="tool0"/>
+    <child  link="ee_mount"/>
+    <!-- Adjust if your STL needs an offset/rotation relative to tool0 -->
+    <origin xyz="0 0 0.10" rpy="0 ${pi} 0"/>
+  </joint>
+</robot>

File: src/end_effector_description/urdf/end_effector_withDriverSupport.xacro (robot description, xacro)
@@ -1,14 +1,15 @@
 <?xml version="1.0"?>
 <robot name="end_effector_withDriverSupport" xmlns:xacro="http://ros.org/wiki/xacro">
-  <!-- === UR arm (set the args the UR xacro expects) === -->
-  <xacro:arg name="name" default="ur5e"/>
-  <xacro:arg name="ur_type" default="ur5e"/>
-  <!-- Use find-pkg-share on ROS 2 -->
-  <xacro:include filename="$(find-pkg-share ur_description)/urdf/ur.urdf.xacro"/>
-  <!-- Instantiate the UR with empty prefix (tool0, flange, etc. will exist) -->
-  <xacro:ur_robot name="$(arg name)" ur_type="$(arg ur_type)" prefix=""/>
-  <!-- === End-effector macro (visual + collision) === -->
-  <xacro:include filename="$(find-pkg-share end_effector_description)/urdf/end_effector.urdf.xacro"/>
-  <!-- Mount the gripper directly to tool0. Adjust pose as needed. -->
+  <!-- UR args (prefer ur5e unless you truly have ur5) -->
+  <xacro:arg name="name"    default="ur5e"/>
+  <xacro:arg name="ur_type" default="ur5"/>
+  <xacro:arg name="prefix"  default=""/>
+  <!-- UR robot -->
+  <xacro:include filename="$(find ur_description)/urdf/ur.urdf.xacro"/>
+  <!-- Don't pass ur_type here; it's consumed internally by ur.urdf.xacro -->
+  <!-- <xacro:ur_robot name="$(arg name)"/> -->
+  <!-- End-effector macro (your file above) -->
+  <xacro:include filename="$(find end_effector_description)/urdf/end_effector.urdf.xacro"/>
+  <!-- Mount the gripper to tool0 -->
   <xacro:end_effector prefix="" parent="tool0"/>
 </robot>
