Commit message: can visualise endeffector

File: src/end_effector_description/urdf/end_effector.urdf (robot description, URDF)
Before this commit: robot simple_claw, 1 links, 0 joints
Links:
- link ee_mount: geometry collision box size=0.06 0.083 0.112; visual mesh filename=package://end_effector_description/meshes/claw_assembly.stl scale=0.001 0.001 0.001

Commit message: confirmed stable

File: src/end_effector_description/urdf/end_effector.urdf (robot description, URDF)
Before this commit: robot end_effector, 1 links, 0 joints
Links:
- link gripper: geometry collision box size=0.06 0.09 0.05; visual mesh filename=package://end_effector_description/meshes/claw_assembly.stl scale=0.001 0.001 0.001
